Commit message: major changed in URDF

File: src/My_Robotv3/urdf/My_Robot_Cam_UDRF.xacro (robot description, xacro)
@@ -141,5 +141,5 @@
   <!-- Joints -->
   <joint name="${prefix}camera_joint" type="fixed">
-    <origin xyz="0.36 0.186 0.344" rpy="0 0 0"/>
+    <origin xyz="0.36 0.186 0.344" rpy="0 -0.34906585 0"/>
     <parent link="${prefix}base_link"/>
     <child link="${prefix}camera_1"/>

Commit message: added urdf caster wheel

File: src/My_Robotv3/urdf/My_Robot_Cam_UDRF.xacro (robot description, xacro)
@@ -118,4 +118,25 @@
       xyz="-0.024 0.2012 0.232" rpy="0 0 0" material_name="silver"/>
   </link>
+  <!-- Caster wheel (mesh-based, template aligned with back files) -->
+  <link name="${prefix}caster_wheel_1">
+    <inertial>
+      <origin xyz="0 0 0" rpy="0 0 0"/>
+      <mass value="0.1"/>
+      <inertia ixx="1e-4" iyy="1e-4" izz="1e-4" ixy="0.0" iyz="0.0" ixz="0.0"/>
+    </inertial>
+    <visual>
+      <origin xyz="0 0 0" rpy="0 0 0"/>
+      <geometry>
+        <mesh filename="file://${mesh_dir}/caster_wheel_1.stl" scale="${mesh_scale}"/>
+      </geometry>
+      <material name="silver"/>
+    </visual>
+    <collision>
+      <origin xyz="0 0 0" rpy="0 0 0"/>
+      <geometry>
+        <mesh filename="file://${mesh_dir}/caster_wheel_1.stl" scale="${mesh_scale}"/>
+      </geometry>
+    </collision>
+  </link>
   <!-- Arms -->
   <link name="${prefix}left_arm_1">
@@ -177,4 +198,9 @@
     <dynamics damping="0.0" friction="0.0"/>
   </joint>
+  <joint name="${prefix}caster_wheel_joint" type="fixed">
+    <origin xyz="-0.8 0 0" rpy="0 0 0"/>
+    <parent link="${prefix}base_link"/>
+    <child link="${prefix}caster_wheel_1"/>
+  </joint>
   <joint name="${prefix}left_arm" type="continuous">
     <origin xyz="-0.033381 0.517012 -0.2155" rpy="0 0 0"/>

Commit message: updated URDF but Still off + Added perception node

File: src/My_Robotv3/urdf/My_Robot_Cam_UDRF.xacro (robot description, xacro)
@@ -53,5 +53,5 @@
   <link name="${prefix}base_link">
     <inertial>
-      <origin xyz="-0.07327696957668513 0.18599999999999897 0.03780217439911652" rpy="0 0 0"/>
+      <origin xyz="-0.09727696957668519 -1.0302869668521452e-15 0.4078021743991166" rpy="0 0 0"/>
       <mass value="234.7770329034331"/>
       <inertia ixx="30.45054" iyy="20.65215" izz="32.896368" ixy="-0.0" iyz="-0.0" ixz="-0.345272"/>
@@ -64,5 +64,5 @@
   <link name="${prefix}camera_1">
     <inertial>
-      <origin xyz="0 0 -0.017" rpy="0 0 0"/>
+      <origin xyz="5.551115123125783e-17 0.0 -0.017000000000000126" rpy="0 0 0"/>
       <mass value="1.191651999466405"/>
       <inertia ixx="0.000907" iyy="0.000363" izz="0.00104" ixy="0.0" iyz="0.0" ixz="0.0"/>
@@ -70,5 +70,5 @@
     <xacro:mesh_visual_collision
       mesh_path="file://${mesh_dir}/camera_1.stl"
-      xyz="-0.36 -0.186 -0.344" rpy="0 0 0" material_name="silver"/>
+      xyz="-0.336 0.0 -0.714" rpy="0 0 0" material_name="silver"/>
   </link>
   <!-- Standard ROS camera optical frame (handy for image pipelines) -->
@@ -82,11 +82,11 @@
   <link name="${prefix}lidar_1">
     <inertial>
-      <origin xyz="0.02 0 -0.007" rpy="0 0 0"/>
+      <origin xyz="0.04399999999999997 0.18599999999999997 -0.3770000000000002" rpy="0 0 0"/>
       <mass value="2.1007654145366375"/>
-      <inertia ixx="0.001356" iyy="0.001356" izz="0.002034" ixy="0.0" iyz="-0.0" ixz="-0.0"/>
+      <inertia ixx="0.001356" iyy="0.001356" izz="0.002034" ixy="0.0" iyz="-0.0" ixz="0.0"/>
     </inertial>
     <xacro:mesh_visual_collision
       mesh_path="file://${mesh_dir}/lidar_1.stl"
-      xyz="-0.002 -0.186 -0.384" rpy="0 0 0" material_name="silver"/>
+      xyz="0.046 0.186 -1.124" rpy="0 0 0" material_name="silver"/>
   </link>
   <link name="${prefix}laser_frame">
@@ -100,5 +100,5 @@
   <link name="${prefix}left_wheel_1">
     <inertial>
-      <origin xyz="0 0.023 -0.03" rpy="0 0 0"/>
+      <origin xyz="0.02400000000000009 0.20900000000000019 -0.4000000000000001" rpy="0 0 0"/>
       <mass value="1.555503053757221"/>
       <inertia ixx="0.004956" iyy="0.009411" izz="0.004956" ixy="0.0" iyz="0.0" ixz="0.0"/>
@@ -106,9 +106,9 @@
     <xacro:mesh_visual_collision
       mesh_path="file://${mesh_dir}/left_wheel_1.stl"
-      xyz="-0.024 -0.5732 0.232" rpy="0 0 0" material_name="silver"/>
+      xyz="0.024 -0.2012 -0.508" rpy="0 0 0" material_name="silver"/>
   </link>
   <link name="${prefix}right_wheel_1">
     <inertial>
-      <origin xyz="0 -0.023 -0.03" rpy="0 0 0"/>
+      <origin xyz="0.023999999999999917 0.1630000000000001 -0.4" rpy="0 0 0"/>
       <mass value="1.5555030537572214"/>
       <inertia ixx="0.004956" iyy="0.009411" izz="0.004956" ixy="0.0" iyz="0.0" ixz="0.0"/>
@@ -116,31 +116,21 @@
     <xacro:mesh_visual_collision
       mesh_path="file://${mesh_dir}/right_wheel_1.stl"
-      xyz="-0.024 0.2012 0.232" rpy="0 0 0" material_name="silver"/>
+      xyz="0.024 0.5732 -0.508" rpy="0 0 0" material_name="silver"/>
   </link>
   <!-- Caster wheel (mesh-based, template aligned with back files) -->
   <link name="${prefix}caster_wheel_1">
     <inertial>
-      <origin xyz="0 0 0" rpy="0 0 0"/>
-      <mass value="0.1"/>
-      <inertia ixx="1e-4" iyy="1e-4" izz="1e-4" ixy="0.0" iyz="0.0" ixz="0.0"/>
-    </inertial>
-    <visual>
-      <origin xyz="0 0 0" rpy="0 0 0"/>
-      <geometry>
-        <mesh filename="file://${mesh_dir}/caster_wheel_1.stl" scale="${mesh_scale}"/>
-      </geometry>
-      <material name="silver"/>
-    </visual>
-    <collision>
-      <origin xyz="0 0 0" rpy="0 0 0"/>
-      <geometry>
-        <mesh filename="file://${mesh_dir}/caster_wheel_1.stl" scale="${mesh_scale}"/>
-      </geometry>
-    </collision>
+      <origin xyz="0.013999999999999957 0.18633913892803772 -0.42461804516587487" rpy="0 0 0"/>
+      <mass value="4.669751850982787"/>
+      <inertia ixx="0.005221" iyy="0.005251" izz="0.008081" ixy="0.0" iyz="-0.0" ixz="0.0"/>
+    </inertial>
+    <xacro:mesh_visual_collision
+      mesh_path="file://${mesh_dir}/caster_wheel_1.stl"
+      xyz="0.365 0.186227 -0.464" rpy="0 0 0" material_name="silver"/>
   </link>
   <!-- Arms -->
   <link name="${prefix}left_arm_1">
     <inertial>
-      <origin xyz="0.1917093322749274 -0.002691315286684093 -0.02" rpy="0 0 0"/>
+      <origin xyz="0.19170933227492737 -0.002691315286684093 -0.020000000000000157" rpy="0 0 0"/>
       <mass value="2.420566632833367"/>
       <inertia ixx="0.000455" iyy="0.031668" izz="0.031478" ixy="0.000981" iyz="-0.0" ixz="0.0"/>
@@ -148,19 +138,19 @@
     <xacro:mesh_visual_collision
       mesh_path="file://${mesh_dir}/left_arm_1.stl"
-      xyz="0.033381 -0.517012 0.2155" rpy="0 0 0" material_name="silver"/>
+      xyz="0.057381 -0.331012 -0.1545" rpy="0 0 0" material_name="silver"/>
   </link>
   <link name="${prefix}right_arm_1">
     <inertial>
-      <origin xyz="0.1917093322749274 0.002692315286683955 -0.02" rpy="0 0 0"/>
+      <origin xyz="0.19170933227492737 0.0026923152866838995 -0.0200000000000001" rpy="0 0 0"/>
       <mass value="2.420566632833367"/>
-      <inertia ixx="0.000455" iyy="0.031668" izz="0.031478" ixy="-0.000981" iyz="0.0" ixz="0.0"/>
+      <inertia ixx="0.000455" iyy="0.031668" izz="0.031478" ixy="-0.000981" iyz="-0.0" ixz="-0.0"/>
     </inertial>
     <xacro:mesh_visual_collision
       mesh_path="file://${mesh_dir}/right_arm_1.stl"
-      xyz="0.033381 0.145013 0.2155" rpy="0 0 0" material_name="silver"/>
+      xyz="0.057381 0.331013 -0.1545" rpy="0 0 0" material_name="silver"/>
   </link>
   <!-- Joints -->
   <joint name="${prefix}camera_joint" type="fixed">
-    <origin xyz="0.36 0.186 0.344" rpy="0 -0.34906585 0"/>
+    <origin xyz="0.336 0.0 0.714" rpy="0 0 0"/>
     <parent link="${prefix}base_link"/>
     <child link="${prefix}camera_1"/>
@@ -173,5 +163,5 @@
   </joint>
   <joint name="${prefix}lidar_joint" type="fixed">
-    <origin xyz="0.002 0.186 0.384" rpy="0 0 0"/>
+    <origin xyz="-0.046 -0.186 1.124" rpy="0 0 0"/>
     <parent link="${prefix}base_link"/>
     <child link="${prefix}lidar_1"/>
@@ -183,5 +173,5 @@
   </joint>
   <joint name="${prefix}left_wheel" type="continuous">
-    <origin xyz="0.024 0.5732 -0.232" rpy="0 0 0"/>
+    <origin xyz="-0.024 0.2012 0.508" rpy="0 0 0"/>
     <parent link="${prefix}base_link"/>
     <child link="${prefix}left_wheel_1"/>
@@ -191,29 +181,29 @@
   </joint>
   <joint name="${prefix}right_wheel" type="continuous">
-    <origin xyz="0.024 -0.2012 -0.232" rpy="0 0 0"/>
+    <origin xyz="-0.024 -0.5732 0.508" rpy="0 0 0"/>
     <parent link="${prefix}base_link"/>
     <child link="${prefix}right_wheel_1"/>
-    <axis xyz="0 -1 0"/>
+    <axis xyz="-0.0 -1.0 0.0"/>
     <limit effort="5.0" velocity="30.0"/>
     <dynamics damping="0.0" friction="0.0"/>
   </joint>
   <joint name="${prefix}caster_wheel_joint" type="fixed">
-    <origin xyz="-0.8 0 0" rpy="0 0 0"/>
+    <origin xyz="-0.365 -0.186227 0.464" rpy="0 0 0"/>
     <parent link="${prefix}base_link"/>
     <child link="${prefix}caster_wheel_1"/>
   </joint>
   <joint name="${prefix}left_arm" type="continuous">
-    <origin xyz="-0.033381 0.517012 -0.2155" rpy="0 0 0"/>
+    <origin xyz="-0.057381 0.331012 0.1545" rpy="0 0 0"/>
     <parent link="${prefix}base_link"/>
     <child link="${prefix}left_arm_1"/>
-    <axis xyz="0 0 -1"/>
+    <axis xyz="-0.0 0.0 -1.0"/>
     <limit effort="2.0" velocity="2.0"/>
     <dynamics damping="0.2" friction="0.1"/>
   </joint>
   <joint name="${prefix}right_arm" type="continuous">
-    <origin xyz="-0.033381 -0.145013 -0.2155" rpy="0 0 0"/>
+    <origin xyz="-0.057381 -0.331013 0.1545" rpy="0 0 0"/>
     <parent link="${prefix}base_link"/>
     <child link="${prefix}right_arm_1"/>
-    <axis xyz="0 0 1"/>
+    <axis xyz="0.0 0.0 1.0"/>
     <limit effort="2.0" velocity="2.0"/>
     <dynamics damping="0.2" friction="0.1"/>

Commit message: added readme

File: src/My_Robotv3/urdf/My_Robot_Cam_UDRF.xacro (robot description, xacro)
@@ -1,13 +1,4 @@
 <?xml version="1.0"?>
 <robot name="my_robot_v3" xmlns:xacro="http://www.ros.org/wiki/xacro">
-  <!--
-    Cleaned / ROS2-friendly Xacro.
-    Notes:
-    - Link meshes appear to be exported in *assembly coordinates* (common from CAD exports).
-      That’s why many links have a non-zero <visual>/<collision> origin that is "cancelled" by
-      the joint origin.
-    - Default names are preserved (base_link, camera_1, lidar_1, ...) so existing RViz configs
-      and launch files keep working.
-  -->
   <!-- Optional prefix for multi-robot use -->
   <xacro:arg name="prefix" default=""/>
@@ -21,4 +12,38 @@
   <xacro:include filename="$(find my_robot_v3_description)/urdf/My_Robot_Cam_UDRF.ros2control"/>
   <xacro:include filename="$(find my_robot_v3_description)/urdf/My_Robot_Cam_UDRF.gazebo"/>
+  <!--
+    ==========================================================
+    POSES (EDIT ONLY HERE)
+    These are the link-frame poses relative to base_link.
+    Visual/collision will automatically use the NEGATIVE values
+    to keep your assembly-exported STLs aligned.
+    ==========================================================
+  -->
+  <!-- camera_1 -->
+  <xacro:property name="cam_x" value="0.336"/>
+  <xacro:property name="cam_y" value="0.0"/>
+  <xacro:property name="cam_z" value="0.714"/>
+  <!-- lidar_1 -->
+  <xacro:property name="lidar_x" value="-0.046"/>
+  <xacro:property name="lidar_y" value="-0.186"/>
+  <xacro:property name="lidar_z" value="1.124"/>
+  <!-- wheels -->
+  <xacro:property name="lw_x" value="-0.024"/>
+  <xacro:property name="lw_y" value="0.2012"/>
+  <xacro:property name="lw_z" value="0.508"/>
+  <xacro:property name="rw_x" value="-0.024"/>
+  <xacro:property name="rw_y" value="-0.5732"/>
+  <xacro:property name="rw_z" value="0.508"/>
+  <!-- caster -->
+  <xacro:property name="caster_x" value="-0.365"/>
+  <xacro:property name="caster_y" value="-0.186227"/>
+  <xacro:property name="caster_z" value="0.464"/>
+  <!-- arms -->
+  <xacro:property name="la_x" value="-0.057381"/>
+  <xacro:property name="la_y" value="0.331012"/>
+  <xacro:property name="la_z" value="0.1545"/>
+  <xacro:property name="ra_x" value="-0.057381"/>
+  <xacro:property name="ra_y" value="-0.331013"/>
+  <xacro:property name="ra_z" value="0.1545"/>
   <!-- Small helper macro to reduce repetition -->
   <xacro:macro name="mesh_visual_collision" params="mesh_path xyz rpy material_name">
@@ -38,5 +63,4 @@
   </xacro:macro>
   <!-- Base -->
-  <!-- base_footprint is commonly expected by Nav2; keep it aligned with base_link for now -->
   <link name="${prefix}base_footprint">
     <inertial>
@@ -61,5 +85,5 @@
       xyz="0 0 0" rpy="0 0 0" material_name="silver"/>
   </link>
-  <!-- Sensors (visual geometry only; Gazebo sensors/plugins can be added in My_Robot_Cam_UDRF.gazebo) -->
+  <!-- Sensors -->
   <link name="${prefix}camera_1">
     <inertial>
@@ -68,9 +92,9 @@
       <inertia ixx="0.000907" iyy="0.000363" izz="0.00104" ixy="0.0" iyz="0.0" ixz="0.0"/>
     </inertial>
+    <!-- NEGATED pose to match assembly-exported STL -->
     <xacro:mesh_visual_collision
       mesh_path="file://${mesh_dir}/camera_1.stl"
-      xyz="-0.336 0.0 -0.714" rpy="0 0 0" material_name="silver"/>
-  </link>
-  <!-- Standard ROS camera optical frame (handy for image pipelines) -->
+      xyz="${-cam_x} ${-cam_y} ${-cam_z}" rpy="0 0 0" material_name="silver"/>
+  </link>
   <link name="${prefix}camera_optical_frame">
     <inertial>
@@ -88,5 +112,5 @@
     <xacro:mesh_visual_collision
       mesh_path="file://${mesh_dir}/lidar_1.stl"
-      xyz="0.046 0.186 -1.124" rpy="0 0 0" material_name="silver"/>
+      xyz="${-lidar_x} ${-lidar_y} ${-lidar_z}" rpy="0 0 0" material_name="silver"/>
   </link>
   <link name="${prefix}laser_frame">
@@ -106,5 +130,5 @@
     <xacro:mesh_visual_collision
       mesh_path="file://${mesh_dir}/left_wheel_1.stl"
-      xyz="0.024 -0.2012 -0.508" rpy="0 0 0" material_name="silver"/>
+      xyz="${-lw_x} ${-lw_y} ${-lw_z}" rpy="0 0 0" material_name="silver"/>
   </link>
   <link name="${prefix}right_wheel_1">
@@ -116,7 +140,7 @@
     <xacro:mesh_visual_collision
       mesh_path="file://${mesh_dir}/right_wheel_1.stl"
-      xyz="0.024 0.5732 -0.508" rpy="0 0 0" material_name="silver"/>
-  </link>
-  <!-- Caster wheel (mesh-based, template aligned with back files) -->
+      xyz="${-rw_x} ${-rw_y} ${-rw_z}" rpy="0 0 0" material_name="silver"/>
+  </link>
+  <!-- Caster -->
   <link name="${prefix}caster_wheel_1">
     <inertial>
@@ -127,5 +151,5 @@
     <xacro:mesh_visual_collision
       mesh_path="file://${mesh_dir}/caster_wheel_1.stl"
-      xyz="0.365 0.186227 -0.464" rpy="0 0 0" material_name="silver"/>
+      xyz="${-caster_x} ${-caster_y} ${-caster_z}" rpy="0 0 0" material_name="silver"/>
   </link>
   <!-- Arms -->
@@ -138,5 +162,5 @@
     <xacro:mesh_visual_collision
       mesh_path="file://${mesh_dir}/left_arm_1.stl"
-      xyz="0.057381 -0.331012 -0.1545" rpy="0 0 0" material_name="silver"/>
+      xyz="${-la_x} ${-la_y} ${-la_z}" rpy="0 0 0" material_name="silver"/>
   </link>
   <link name="${prefix}right_arm_1">
@@ -148,9 +172,9 @@
     <xacro:mesh_visual_collision
       mesh_path="file://${mesh_dir}/right_arm_1.stl"
-      xyz="0.057381 0.331013 -0.1545" rpy="0 0 0" material_name="silver"/>
+      xyz="${-ra_x} ${-ra_y} ${-ra_z}" rpy="0 0 0" material_name="silver"/>
   </link>
   <!-- Joints -->
   <joint name="${prefix}camera_joint" type="fixed">
-    <origin xyz="0.336 0.0 0.714" rpy="0 0 0"/>
+    <origin xyz="${cam_x} ${cam_y} ${cam_z}" rpy="0 0 0"/>
     <parent link="${prefix}base_link"/>
     <child link="${prefix}camera_1"/>
@@ -163,5 +187,5 @@
   </joint>
   <joint name="${prefix}lidar_joint" type="fixed">
-    <origin xyz="-0.046 -0.186 1.124" rpy="0 0 0"/>
+    <origin xyz="${lidar_x} ${lidar_y} ${lidar_z}" rpy="0 0 0"/>
     <parent link="${prefix}base_link"/>
     <child link="${prefix}lidar_1"/>
@@ -173,5 +197,5 @@
   </joint>
   <joint name="${prefix}left_wheel" type="continuous">
-    <origin xyz="-0.024 0.2012 0.508" rpy="0 0 0"/>
+    <origin xyz="${lw_x} ${lw_y} ${lw_z}" rpy="0 0 0"/>
     <parent link="${prefix}base_link"/>
     <child link="${prefix}left_wheel_1"/>
@@ -181,29 +205,29 @@
   </joint>
   <joint name="${prefix}right_wheel" type="continuous">
-    <origin xyz="-0.024 -0.5732 0.508" rpy="0 0 0"/>
+    <origin xyz="${rw_x} ${rw_y} ${rw_z}" rpy="0 0 0"/>
     <parent link="${prefix}base_link"/>
     <child link="${prefix}right_wheel_1"/>
-    <axis xyz="-0.0 -1.0 0.0"/>
+    <axis xyz="0 -1 0"/>
     <limit effort="5.0" velocity="30.0"/>
     <dynamics damping="0.0" friction="0.0"/>
   </joint>
   <joint name="${prefix}caster_wheel_joint" type="fixed">
-    <origin xyz="-0.365 -0.186227 0.464" rpy="0 0 0"/>
+    <origin xyz="${caster_x} ${caster_y} ${caster_z}" rpy="0 0 0"/>
     <parent link="${prefix}base_link"/>
     <child link="${prefix}caster_wheel_1"/>
   </joint>
   <joint name="${prefix}left_arm" type="continuous">
-    <origin xyz="-0.057381 0.331012 0.1545" rpy="0 0 0"/>
+    <origin xyz="${la_x} ${la_y} ${la_z}" rpy="0 0 0"/>
     <parent link="${prefix}base_link"/>
     <child link="${prefix}left_arm_1"/>
-    <axis xyz="-0.0 0.0 -1.0"/>
+    <axis xyz="0 0 -1"/>
     <limit effort="2.0" velocity="2.0"/>
     <dynamics damping="0.2" friction="0.1"/>
   </joint>
   <joint name="${prefix}right_arm" type="continuous">
-    <origin xyz="-0.057381 -0.331013 0.1545" rpy="0 0 0"/>
+    <origin xyz="${ra_x} ${ra_y} ${ra_z}" rpy="0 0 0"/>
     <parent link="${prefix}base_link"/>
     <child link="${prefix}right_arm_1"/>
-    <axis xyz="0.0 0.0 1.0"/>
+    <axis xyz="0 0 1"/>
     <limit effort="2.0" velocity="2.0"/>
     <dynamics damping="0.2" friction="0.1"/>
